File: picsil Carrier.brd (EAGLE design)
At the start: 91.4 x 54.3 mm, 43 parts, among them IC1 NAND, J1 STX-3120-3BM, J2 STX-3120-3BM, J3 STX-3120-3BM, J5 S2B-PH-SM4-TB(LF)(SN), J6 47346-1001, Q1 MMBT2222A, U1 MB85RC256VPF-G-JNERE2, U11 BORON, U2 TPL5010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

Commit message: updated brd
Parts:
- moved C4 1.26 mm to (74.1, 19.1)
- moved V1 0.79 mm to (82.1, 17.8)
Changed lines of the file:
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@@
 <attribute name="VALUE" x="63.754" y="18.923" size="0.4064" layer="27"/>
 </element>
-<element name="C4" library="MF_Passives" package="CP10MM" value="470uF" x="73.66" y="20.32" smashed="yes" rot="R180">
-<attribute name="HOUSEPART" value="" x="30.48" y="27.94" size="1.778" layer="27" rot="R180" display="off"/>
-<attribute name="MPN" value="" x="30.48" y="27.94" size="1.778" layer="27" rot="R180" display="off"/>
-<attribute name="NAME" x="78.81" y="14.09" size="1.016" layer="25" font="vector" ratio="16" rot="R180"/>
-<attribute name="POPULATE" value="1" x="30.48" y="27.94" size="1.778" layer="27" rot="R180" display="off"/>
-<attribute name="TOLERANCE" value="" x="30.48" y="27.94" size="1.778" layer="27" rot="R180" display="off"/>
-<attribute name="URL" value="" x="30.48" y="27.94" size="1.778" layer="27" rot="R180" display="off"/>
-<attribute name="VOLTAGE" value="" x="30.48" y="27.94" size="1.778" layer="27" rot="R180" display="off"/>
+<element name="C4" library="MF_Passives" package="CP10MM" value="470uF" x="74.056875" y="19.129375" smashed="yes" rot="R180">
+<attribute name="HOUSEPART" value="" x="30.876875" y="26.749375" size="1.778" layer="27" rot="R180" display="off"/>
+<attribute name="MPN" value="" x="30.876875" y="26.749375" size="1.778" layer="27" rot="R180" display="off"/>
+<attribute name="NAME" x="79.206875" y="12.899375" size="1.016" layer="25" font="vector" ratio="16" rot="R180"/>
+<attribute name="POPULATE" value="1" x="30.876875" y="26.749375" size="1.778" layer="27" rot="R180" display="off"/>
+<attribute name="TOLERANCE" value="" x="30.876875" y="26.749375" size="1.778" layer="27" rot="R180" display="off"/>
+<attribute name="URL" value="" x="30.876875" y="26.749375" size="1.778" layer="27" rot="R180" display="off"/>
+<attribute name="VOLTAGE" value="" x="30.876875" y="26.749375" size="1.778" layer="27" rot="R180" display="off"/>
 </element>
 <element name="D1" library="MF_Discrete_Semiconductor" package="SOD-123" value="MF-DIO-SOD123-BAT42" x="38.1" y="21.59" smashed="yes" rot="R180">
@@
 <attribute name="MOUSER_PART_NUMBER" value="612-TL1105S-250" x="101.6" y="-109.22" size="1.778" layer="27" display="off"/>
 <attribute name="MOUSER_PRICE-STOCK" value="https://www.mouser.com/Search/Refine.aspx?Keyword=612-TL1105S-250" x="101.6" y="-109.22" size="1.778" layer="27" display="off"/>
-<attribute name="NAME" x="78.74" y="11.43" size="1.27" layer="25" align="center"/>
+<attribute name="NAME" x="79.930625" y="9.445625" size="1.27" layer="25" align="center"/>
 <attribute name="VALUE" x="81.28" y="5.08" size="1.27" layer="27" align="center"/>
 </element>
@@
 <attribute name="PRICE" value="None" x="74.93" y="-41.91" size="1.778" layer="27" display="off"/>
 </element>
-<element name="V1" library="Custom Components" package="0805" value="VC080505C150DP " x="81.28" y="17.78" smashed="yes" rot="R90">
-<attribute name="NAME" x="80.3148" y="17.78" size="0.8128" layer="25" font="vector" rot="R90" align="bottom-center"/>
-<attribute name="VALUE" x="82.2452" y="17.78" size="0.8128" layer="27" font="vector" rot="R90" align="top-center"/>
+<element name="V1" library="Custom Components" package="0805" value="VC080505C150DP " x="82.07375" y="17.78" smashed="yes" rot="R90">
+<attribute name="NAME" x="81.10855" y="17.78" size="0.8128" layer="25" font="vector" rot="R90" align="bottom-center"/>
+<attribute name="VALUE" x="83.03895" y="17.78" size="0.8128" layer="27" font="vector" rot="R90" align="top-center"/>
 </element>
 <element name="V3" library="Custom Components" package="0805" value="VC080505C150DP " x="33.02" y="19.05" smashed="yes">
@@
 <via x="85.09" y="12.7" extent="1-16" drill="0.35"/>
 <via x="81.28" y="11.43" extent="1-16" drill="0.35"/>
-<via x="76.2" y="13.97" extent="1-16" drill="0.35"/>
-<via x="69.85" y="13.97" extent="1-16" drill="0.35"/>
+<via x="76.2" y="11.58875" extent="1-16" drill="0.35"/>
+<via x="69.85" y="11.58875" extent="1-16" drill="0.35"/>
 <via x="63.5" y="13.97" extent="1-16" drill="0.35"/>
 <via x="73.66" y="7.62" extent="1-16" drill="0.35"/>
@@
 <wire x1="77.47" y1="50.8" x2="76.2" y2="52.07" width="0.508" layer="1"/>
 <wire x1="76.2" y1="52.07" x2="44.45" y2="52.07" width="0.508" layer="1"/>
-<wire x1="73.66" y1="24.67" x2="76.74" y2="24.67" width="0.508" layer="1"/>
-<wire x1="81.28" y1="18.6817" x2="76.74" y2="23.2217" width="0.508" layer="1"/>
-<wire x1="76.74" y1="23.2217" x2="76.74" y2="24.67" width="0.508" layer="1"/>
+<wire x1="74.056875" y1="23.479375" x2="76.74" y2="23.479375" width="0.508" layer="1"/>
+<wire x1="82.07375" y1="18.6817" x2="76.74" y2="24.01545" width="0.508" layer="1"/>
+<wire x1="76.74" y1="23.479375" x2="76.74" y2="24.01545" width="0.508" layer="1"/>
+<wire x1="76.74" y1="24.01545" x2="76.74" y2="24.67" width="0.508" layer="1"/>
 <wire x1="82.7225" y1="22.780625" x2="80.01" y2="22.780625" width="0.508" layer="1"/>
 <wire x1="44.45" y1="52.07" x2="41.91" y2="49.53" width="0.508" layer="1"/>

Commit message: mounting holes and fiducials
Parts:
- added H2, H3, H4, H5: MOUNT-HOLE3.2, holes:3,2
- added U$1, U$2, U$3, U$4: FIDUCIAL, adafruit:FIDUCIAL_1MM
- moved S1 3.57 mm to (77.7, 5.08)
- moved J6 0.40 mm to (92.1, 31.3)
Routing:
- net N$24: track 9.98 -> 6.53 mm
- net N$25: track 42.1 -> 40.0 mm
Other:
- board size 91.4 x 54.3 mm -> 95 x 54.3 mm
- board text added: "+"
- board text added: "LIPO BAT"
- board text added: "picsil Sense P2 Rev A"

Commit message: finalized Rev A
Parts:
- added FRAME4: FRAME-LETTER, SparkFun-Aesthetics:CREATIVE_COMMONS
- moved FRAME1 26.3 mm to (-73.4, -12.3)
Other:
- board text added: "CS DC RST MOSI SCK VCC GND"
Changed lines of the file:
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@@
 <text x="1.984375" y="26.19375" size="1.778" layer="25">picsil Sense
 P2 Rev A</text>
+<text x="45.640625" y="21.43125" size="0.8128" layer="25">CS  DC  RST MOSI SCK VCC GND</text>
+<text x="16.271875" y="50.8" size="1.778" layer="25">+</text>
 </plain>
 <attributes>
@@
 <attribute name="VALUE" x="33.02" y="34.417" size="0.6096" layer="27" font="vector" ratio="20" align="top-center"/>
 </element>
-<element name="FRAME1" library="SparkFun-Aesthetics" library_urn="urn:adsk.eagle:library:507" package="CREATIVE_COMMONS" package3d_urn="urn:adsk.eagle:package:37121/1" value="FRAME-LETTER" x="-73.66" y="13.97" smashed="yes">
-<attribute name="_EXTERNAL_" value="1" x="-73.66" y="13.97" size="1.778" layer="27" display="off"/>
-</element>
 <element name="FRAME2" library="SparkFun-Aesthetics" library_urn="urn:adsk.eagle:library:507" package="CREATIVE_COMMONS" package3d_urn="urn:adsk.eagle:package:37121/1" value="FRAME-LETTER" x="-73.66" y="25.4" smashed="yes"/>
 <element name="FRAME3" library="SparkFun-Aesthetics" library_urn="urn:adsk.eagle:library:507" package="CREATIVE_COMMONS" package3d_urn="urn:adsk.eagle:package:37121/1" value="FRAME-LETTER" x="-72.39" y="35.56" smashed="yes"/>
@@
 <attribute name="MF" value="" x="100.33" y="-88.9" size="1.778" layer="27" display="off"/>
 <attribute name="MPN" value="" x="100.33" y="-88.9" size="1.778" layer="27" display="off"/>
-<attribute name="NAME" x="44.45" y="25.781" size="1.27" layer="25" ratio="10"/>
+<attribute name="NAME" x="42.06875" y="23.796625" size="1.27" layer="25" ratio="10"/>
 <attribute name="OC_FARNELL" value="unknown" x="100.33" y="-88.9" size="1.778" layer="27" display="off"/>
 <attribute name="OC_NEWARK" value="unknown" x="100.33" y="-88.9" size="1.778" layer="27" display="off"/>
@@
 <element name="J5" library="SparkFun-Connectors" package="JST-2-SMD" value="S2B-PH-SM4-TB(LF)(SN)" x="11.43" y="49.53" smashed="yes">
 <attribute name="MFG" value="S2B-PH-SM4-TB(LF)(SN)" x="34.29" y="-29.21" size="1.778" layer="27" display="off"/>
-<attribute name="NAME" x="4.953" y="51.308" size="0.6096" layer="25" font="vector" ratio="20"/>
+<attribute name="NAME" x="5.349875" y="51.308" size="0.6096" layer="25" font="vector" ratio="20"/>
 <attribute name="PROD_ID" value="CONN-11443" x="34.29" y="-29.21" size="1.778" layer="27" display="off"/>
 <attribute name="SF_ID" value="PRT-08612" x="34.29" y="-29.21" size="1.778" layer="27" display="off"/>
@@
 <element name="H4" library="holes" library_urn="urn:adsk.eagle:library:237" package="3,2" package3d_urn="urn:adsk.eagle:package:14275/1" value="MOUNT-HOLE3.2" x="0.79375" y="50.00625" smashed="yes"/>
 <element name="H5" library="holes" library_urn="urn:adsk.eagle:library:237" package="3,2" package3d_urn="urn:adsk.eagle:package:14275/1" value="MOUNT-HOLE3.2" x="87.3125" y="4.365625" smashed="yes"/>
+<element name="FRAME1" library="SparkFun-Aesthetics" library_urn="urn:adsk.eagle:library:507" package="CREATIVE_COMMONS" package3d_urn="urn:adsk.eagle:package:37121/1" value="FRAME-LETTER" x="-73.421875" y="-12.303125" smashed="yes"/>
+<element name="FRAME4" library="SparkFun-Aesthetics" library_urn="urn:adsk.eagle:library:507" package="CREATIVE_COMMONS" package3d_urn="urn:adsk.eagle:package:37121/1" value="FRAME-LETTER" x="-73.421875" y="-21.034375" smashed="yes"/>
 </elements>
 <signals>
